File: DRV8243-breakout/DRV8243-breakout.kicad_sch (KiCad schematic)
At the start: 27 parts, among them J1 Vin, J2 Motor_Output, J3 Conn_01x11_Pin, J4 Motor_Output, Q1 PMOS-AOD409, U1 PDRV8243HRXYQ1, U2 PDRV8243HRXYQ1

Commit message: Some more routing
Connections:
- net OUT1: now also J2.2 (Pin_2); no longer J2.1 (Pin_1)
- net OUT2: now also J2.1 (Pin_1); no longer J2.2 (Pin_2)
- net OUT3: now also J4.2 (Pin_2); no longer J4.1 (Pin_1)
- net OUT4: now also J4.1 (Pin_1); no longer J4.2 (Pin_2)
Changed lines of the file:
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@@
-	(wire
-		(pts
-			(xy 41.91 85.09) (xy 45.72 85.09)
-		)
-		(stroke
-			(width 0)
-			(type default)
-		)
-	)
 	(wire
 		(pts
@@
 	(wire
 		(pts
-			(xy 41.91 93.98) (xy 45.72 93.98)
-		)
-		(stroke
-			(width 0)
-			(type default)
-		)
-	)
-	(wire
-		(pts
 			(xy 167.64 43.18) (xy 168.91 43.18)
 		)
@@
 	(wire
 		(pts
-			(xy 41.91 96.52) (xy 45.72 96.52)
-		)
-		(stroke
-			(width 0)
-			(type default)
-		)
-	)
-	(wire
-		(pts
 			(xy 63.5 160.02) (xy 63.5 161.29)
 		)
@@
 		(pts
 			(xy 226.06 53.34) (xy 237.49 53.34)
-		)
-		(stroke
-			(width 0)
-			(type default)
-		)
-	)
-	(wire
-		(pts
-			(xy 41.91 82.55) (xy 45.72 82.55)
 		)
 		(stroke
@@
 	(global_label "OUT1"
 		(shape input)
-		(at 41.91 82.55 180)
-		(fields_autoplaced yes)
-		(effects
-			(font
-				(size 1.27 1.27)
-			)
-			(justify right)
-		)
-		(property "Intersheetrefs" "${INTERSHEET_REFS}"
-			(at 34.0867 82.55 0)
+		(at 45.72 85.09 180)
+		(fields_autoplaced yes)
+		(effects
+			(font
+				(size 1.27 1.27)
+			)
+			(justify right)
+		)
+		(property "Intersheetrefs" "${INTERSHEET_REFS}"
+			(at 37.8967 85.09 0)
 			(effects
 				(font
@@
 	(global_label "OUT3"
 		(shape input)
-		(at 41.91 93.98 180)
-		(fields_autoplaced yes)
-		(effects
-			(font
-				(size 1.27 1.27)
-			)
-			(justify right)
-		)
-		(property "Intersheetrefs" "${INTERSHEET_REFS}"
-			(at 34.0867 93.98 0)
+		(at 45.72 96.52 180)
+		(fields_autoplaced yes)
+		(effects
+			(font
+				(size 1.27 1.27)
+			)
+			(justify right)
+		)
+		(property "Intersheetrefs" "${INTERSHEET_REFS}"
+			(at 37.8967 96.52 0)
 			(effects
 				(font
@@
 	(global_label "OUT2"
 		(shape input)
-		(at 41.91 85.09 180)
-		(fields_autoplaced yes)
-		(effects
-			(font
-				(size 1.27 1.27)
-			)
-			(justify right)
-		)
-		(property "Intersheetrefs" "${INTERSHEET_REFS}"
-			(at 34.0867 85.09 0)
+		(at 45.72 82.55 180)
+		(fields_autoplaced yes)
+		(effects
+			(font
+				(size 1.27 1.27)
+			)
+			(justify right)
+		)
+		(property "Intersheetrefs" "${INTERSHEET_REFS}"
+			(at 37.8967 82.55 0)
 			(effects
 				(font
@@
 	(global_label "OUT4"
 		(shape input)
-		(at 41.91 96.52 180)
-		(fields_autoplaced yes)
-		(effects
-			(font
-				(size 1.27 1.27)
-			)
-			(justify right)
-		)
-		(property "Intersheetrefs" "${INTERSHEET_REFS}"
-			(at 34.0867 96.52 0)
-			(effects
-				(font
+		(at 45.72 93.98 180)
+		(fields_autoplaced yes)
+		(effects
+			(font
+				(size 1.27 1.27)
+			)
+			(justify right)
+		)
+		(property "Intersheetrefs" "${INTERSHEET_REFS}"
+			(at 37.8967 93.98 0)
+			(effects
+				(font

Commit message: Routing v2
Parts:
- removed J3: Conn_01x11_Pin, Connector_PinHeader_2.54mm:PinHeader_1x11_P2.54mm_Vertical, symbol Connector:Conn_01x11_Pin
- added J3: Conn_02x06_Odd_Even, Connector_PinSocket_2.54mm:PinSocket_2x06_P2.54mm_Vertical, symbol Connector_Generic:Conn_02x06_Odd_Even
Connections:
- net DRVOFF: now also J3.4 (Pin_4)
- net GND: now also J3.1 (Pin_1)
- net IN1: now also J3.9 (Pin_9)
- net IN2: now also J3.7 (Pin_7)
- net IN3: now also J3.10 (Pin_10)
- net IN4: now also J3.8 (Pin_8)
- net IPROPI0: now also J3.11 (Pin_11)
- net IPROPI1: now also J3.12 (Pin_12)
- net Vcc: now also J3.3 (Pin_3)
- net nSLEEP: now also J3.2 (Pin_2)
- net nFault renamed nFault0
- net nFault0: now also J3.5 (Pin_5); no longer R9.2, U2.1 (FAULT_N)
- new net nFault1: J3.6 (Pin_6), R9.2, U2.1 (FAULT_N)

Commit message: Footprint
Parts:
- J3: footprint Connector_PinSocket_2.54mm:PinSocket_2x06_P2.54mm_Vertical -> Connector_PinHeader_2.54mm:PinHeader_1x11_P2.54mm_Vertical
Changed lines of the file:
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@@
 			)
 		)
-		(property "Footprint" "Connector_PinSocket_2.54mm:PinSocket_2x06_P2.54mm_Vertical"
+		(property "Footprint" "Connector_PinHeader_2.54mm:PinHeader_1x11_P2.54mm_Vertical"
 			(at 110.49 48.26 0)
 			(effects
